File: hardware/kicad/tdm-dash.kicad_sch (KiCad schematic)
At the start: 0 parts

Commit message: Schematic: backlight breakout off the board, harness fuse, micro-USB plug
The perfboard has no room for the TPS61169 breakout, and the build steps
already wired it off the board: J701 now gives it +5 V, CTRL and ground,
and its output goes to the panel LED pins (J704), in a dashed box like the
buttons. F101 is marked as the inline fuse of the adapter harness, J401 as
the terminal for the sensor cable, and J703 has the five pins of the
micro-USB plug, with ID tied to ground.

Co-Authored-By: Claude Opus 5.5 <noreply@anthropic.com>
Claude-Session: https://claude.ai/code/session_01G9D4Wshjz9MkaThp4wsrGP
Other:
- note added: "1 Power: bike connectors J101 and J102, harness fuse, reverse polarity, TVS, LC filter, 5 V buck, Pico hold-up 2 Warning lights: neutral, high beam, turn signals and illumination through EL817 optocouplers 3 Tachometer: coil negative to the H11L1 Schmitt trigger 4 Wheel sensor: LJ12A3 inductive sensor on J401, through an EL817 5 Analog inputs: battery voltage, coolant sender and ambient light to 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"
- note added: "J101, J102: bike harness harness fuse, reverse polarity, TVS, LC filter, 5 V buck, Pico hold-up"
- note removed: "1 Power: bike connectors J101 and J102, fuse, reverse polarity, TVS, LC filter, 5 V buck, Pico hold-up 2 Warning lights: neutral, high beam, turn signals and illumination through EL817 optocouplers 3 Tachometer: coil negative to the H11L1 Schmitt trigger 4 Wheel sensor: LJ12A3 inductive sensor on J401, through an EL817 5 Analog inputs: battery voltage, coolant sender and ambient light to the ADC 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"
- note removed: "J101, J102: bike harness fuse, reverse polarity, TVS, LC filter, 5 V buck, Pico hold-up"
Changed lines of the file:
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@@
 		)
 	)
-	(text "J101, J102: bike harness\nfuse, reverse polarity,\nTVS, LC filter, 5 V buck,\nPico hold-up"
+	(text "J101, J102: bike harness\nharness fuse, reverse\npolarity, TVS, LC filter,\n5 V buck, Pico hold-up"
 		(exclude_from_sim no)
 		(at 20.32 99.06 0)
@@
 		)
 	)
-	(text "1 Power: bike connectors J101 and J102, fuse, reverse polarity, TVS, LC filter, 5 V buck, Pico hold-up\n2 Warning lights: neutral, high beam, turn signals and illumination through EL817 optocouplers\n3 Tachometer: coil negative to the H11L1 Schmitt trigger\n4 Wheel sensor: LJ12A3 inductive sensor on J401, through an EL817\n5 Analog inputs: battery voltage, coolant sender and ambient light to the ADC\n6 MCU: Raspberry Pi Pico, FRAM for the odometer, MODE and SET buttons\n7 Backlight and Pi: TPS61169 backlight driver dimmed by the Pico, USB link to the Pi\n8 Backup LEDs: indicators wired straight to the bike, alive with the electronics off"
+	(text "1 Power: bike connectors J101 and J102, harness fuse, reverse polarity, TVS, LC filter, 5 V buck, Pico hold-up\n2 Warning lights: neutral, high beam, turn signals and illumination through EL817 optocouplers\n3 Tachometer: coil negative to the H11L1 Schmitt trigger\n4 Wheel sensor: LJ12A3 inductive sensor on J401, through an EL817\n5 Analog inputs: battery voltage, coolant sender and ambient light to the ADC\n6 MCU: Raspberry Pi Pico, FRAM for the odometer, MODE and SET buttons\n7 Backlight and Pi: TPS61169 backlight driver dimmed by the Pico, USB link to the Pi\n8 Backup LEDs: indicators wired straight to the bike, alive with the electronics off"
 		(exclude_from_sim no)
 		(at 19.05 160.782 0)
